File: hajo/kicad/hajo_idealisdioda/hajo_idealisdioda.kicad_pcb (KiCad board)
At the start: 2 copper layers, 51.1 x 80 mm, 16 parts, among them J1 LEDs, J2 Control, J3 Light switch

Commit message: small pcb fixes
Parts:
- U1: value ~ -> LTC4355
Connections:
- U1 pad 13: unconnected-(U1-~{FUSEFLT2}-Pad13) -> GND
- U1 pad 14: unconnected-(U1-~{FUSEFLT1}-Pad14) -> GND
Routing:
- net GND: track 84.6 -> 98.6 mm
Changed lines of the file:
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@@
   (net 21 "unconnected-(U1-NC-Pad5)")
   (net 22 "unconnected-(U1-SET-Pad10)")
-  (net 23 "unconnected-(U1-~{FUSEFLT2}-Pad13)")
-  (net 24 "unconnected-(U1-~{FUSEFLT1}-Pad14)")
-  (net 25 "unconnected-(RV1-Pad3)")
+  (net 23 "unconnected-(RV1-Pad3)")
   (footprint "Connector_PinHeader_2.54mm:PinHeader_1x02_P2.54mm_Vertical" (layer "F.Cu")
     (at 53.639 33.319 -90)
@@
       (net 16 "Net-(U1-MON1)") (pinfunction "2") (pintype "passive"))
     (pad "3" thru_hole oval (at 0 5.08 90) (size 1.7 1.7) (drill 1) (layers "*.Cu" "*.Mask")
-      (net 25 "unconnected-(RV1-Pad3)") (pinfunction "3") (pintype "passive+no_connect"))
+      (net 23 "unconnected-(RV1-Pad3)") (pinfunction "3") (pintype "passive+no_connect"))
     (model "${KICAD6_3DMODEL_DIR}/Connector_PinHeader_2.54mm.3dshapes/PinHeader_1x03_P2.54mm_Vertical.wrl"
       (offset (xyz 0 0 0))
@@
         (effects (font (size 1 1) (thickness 0.15)))
     )
-    (fp_text value "~" (at 3.81 20.11) (layer "F.Fab")
+    (fp_text value "LTC4355" (at 3.81 20.11) (layer "F.Fab")
         (effects (font (size 1 1) (thickness 0.15)))
     )
@@
       (net 9 "Net-(J1-Pin_4)") (pinfunction "~{PWRFLT2}") (pintype "open_collector"))
     (pad "13" thru_hole oval (at 7.62 7.62) (size 2.4 1.6) (drill 0.8) (layers "*.Cu" "*.Mask")
-      (net 23 "unconnected-(U1-~{FUSEFLT2}-Pad13)") (pinfunction "~{FUSEFLT2}") (pintype "open_collector+no_connect"))
+      (net 1 "GND") (pinfunction "~{FUSEFLT2}") (pintype "open_collector"))
     (pad "14" thru_hole oval (at 7.62 5.08) (size 2.4 1.6) (drill 0.8) (layers "*.Cu" "*.Mask")
-      (net 24 "unconnected-(U1-~{FUSEFLT1}-Pad14)") (pinfunction "~{FUSEFLT1}") (pintype "open_collector+no_connect"))
+      (net 1 "GND") (pinfunction "~{FUSEFLT1}") (pintype "open_collector"))
     (pad "15" thru_hole oval (at 7.62 2.54) (size 2.4 1.6) (drill 0.8) (layers "*.Cu" "*.Mask")
       (net 11 "Net-(J1-Pin_6)") (pinfunction "~{PWRFLT1}") (pintype "open_collector"))
@@
   (segment (start 37.823 78.445) (end 39.888 80.51) (width 1) (layer "B.Cu") (net 1))
   (segment (start 37.383 72.991) (end 37.383 78.005) (width 1) (layer "B.Cu") (net 1))
+  (segment (start 57 67.65) (end 58.525 69.175) (width 0.25) (layer "B.Cu") (net 1))
   (segment (start 44.749 33.319) (end 45.62 34.19) (width 0.25) (layer "B.Cu") (net 1))
   (segment (start 39.888 80.51) (end 54.3 80.51) (width 1) (layer "B.Cu") (net 1))
@@
   (segment (start 27.536 82.89) (end 31.981 78.445) (width 1) (layer "B.Cu") (net 1))
   (segment (start 45.62 34.19) (end 45.62 47.754991) (width 0.25) (layer "B.Cu") (net 1))
+  (segment (start 58.525 69.175) (end 58.525 76.285) (width 0.25) (layer "B.Cu") (net 1))
   (segment (start 39.323 63.472679) (end 39.323 71.051) (width 1) (layer "B.Cu") (net 1))
+  (segment (start 58.525 76.285) (end 57 77.81) (width 0.25) (layer "B.Cu") (net 1))
   (segment (start 36.769001 56.384999) (end 36.769001 60.91868) (width 1) (layer "B.Cu") (net 1))
   (segment (start 31.981 78.445) (end 37.823 78.445) (width 1) (layer "B.Cu") (net 1))
   (segment (start 37.383 78.005) (end 37.823 78.445) (width 1) (layer "B.Cu") (net 1))
+  (segment (start 57 65.11) (end 57 67.65) (width 0.25) (layer "B.Cu") (net 1))
   (segment (start 27.536 67.65) (end 49.38 67.65) (width 1) (layer "F.Cu") (net 2))
   (segment (start 22.719 29.976) (end 53.199 29.976) (width 1) (layer "F.Cu") (net 2))

Commit message: fix boards
Parts:
- added J4: Light switch, Connector_PinHeader_2.54mm:PinHeader_1x02_P2.54mm_Vertical, F.Cu at (54.4, 39.2)
- moved R2 2.13 mm to (47.3, 56.1)
- moved R3 2.13 mm to (47.5, 70.7)
- moved R4 2.13 mm to (47.5, 79.0)
- moved R6 2.13 mm to (39.2, 47.8)
- moved R7 2.13 mm to (43.0, 47.8)
- moved R8 2.13 mm to (46.6, 47.8)
- moved J2 2.13 mm to (29.6, 83.4)
- moved J1 2.13 mm to (29.0, 33.8)
- moved R1 2.13 mm to (47.4, 64.5)
- moved R5 2.13 mm to (35.6, 47.8)
- moved RV3 2.13 mm to (41.2, 74.9)
- moved U1 2.13 mm to (51.4, 60.6)
- moved RV1 2.13 mm to (41.2, 60.3)
- moved J3 0.94 mm to (54.4, 33.9)
Routing:
- net Net-(J2-Pin_4): track 96.2 -> 100.3 mm
- net Net-(J3-Pin_2): track 27.6 -> 27.1 mm
Other:
- outline, holes or cut-outs redrawn
- board text added: "+"
- board text added: "-"
