File: hajo/kicad/hajo_idealisdioda/hajo_idealisdioda.kicad_sch (KiCad schematic)
At the start: 16 parts, among them J1 LEDs, J2 Control, J3 Light switch

Commit message: small pcb fixes
Parts:
- U1: value ~ -> LTC4355
Connections:
- net GND: now also U1.13 (~{FUSEFLT2}), U1.14 (~{FUSEFLT1})
- no-connect marks 5 -> 3
Changed lines of the file:
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@@
 (kicad_sch (version 20230121) (generator eeschema)
   (paper "A4")
+  (junction (at 120.65 72.39) (diameter 0) (color 0 0 0 0)
+  )
   (junction (at 73.66 43.18) (diameter 0) (color 0 0 0 0)
   )
@@
   )
   (junction (at 92.71 30.48) (diameter 0) (color 0 0 0 0)
+  )
+  (junction (at 143.51 59.69) (diameter 0) (color 0 0 0 0)
   )
   (junction (at 55.88 30.48) (diameter 0) (color 0 0 0 0)
@@
   (no_connect (at 105.41 58.42))
   (no_connect (at 77.47 48.26))
-  (no_connect (at 142.24 59.69))
-  (no_connect (at 142.24 57.15))
   (no_connect (at 77.47 30.48))
   (wire (pts (xy 170.18 27.94) (xy 173.99 27.94))
@@
     (stroke (width 0) (type default))
   )
+  (wire (pts (xy 143.51 72.39) (xy 120.65 72.39))
+    (stroke (width 0) (type default))
+  )
   (wire (pts (xy 104.14 30.48) (xy 104.14 52.07))
     (stroke (width 0) (type default))
@@
     (stroke (width 0) (type default))
   )
+  (wire (pts (xy 143.51 57.15) (xy 143.51 59.69))
+    (stroke (width 0) (type default))
+  )
   (wire (pts (xy 160.02 38.1) (xy 162.56 38.1))
     (stroke (width 0) (type default))
@@
     (stroke (width 0) (type default))
   )
+  (wire (pts (xy 142.24 57.15) (xy 143.51 57.15))
+    (stroke (width 0) (type default))
+  )
   (wire (pts (xy 147.32 64.77) (xy 147.32 43.18))
     (stroke (width 0) (type default))
@@
     (stroke (width 0) (type default))
   )
+  (wire (pts (xy 120.65 72.39) (xy 120.65 73.66))
+    (stroke (width 0) (type default))
+  )
   (wire (pts (xy 73.66 26.67) (xy 73.66 24.13))
     (stroke (width 0) (type default))
@@
     (stroke (width 0) (type default))
   )
-  (wire (pts (xy 120.65 69.85) (xy 120.65 73.66))
+  (wire (pts (xy 120.65 69.85) (xy 120.65 72.39))
     (stroke (width 0) (type default))
   )
@@
     (stroke (width 0) (type default))
   )
+  (wire (pts (xy 143.51 59.69) (xy 143.51 72.39))
+    (stroke (width 0) (type default))
+  )
   (wire (pts (xy 170.18 38.1) (xy 184.15 38.1))
     (stroke (width 0) (type default))
@@
   )
   (wire (pts (xy 73.66 43.18) (xy 91.44 43.18))
+    (stroke (width 0) (type default))
+  )
+  (wire (pts (xy 142.24 59.69) (xy 143.51 59.69))
     (stroke (width 0) (type default))
   )
@@
       (effects (font (size 1.27 1.27)))
     )
-    (property "Value" "~" (at 99.06 74.93 0)
+    (property "Value" "LTC4355" (at 99.06 74.93 0)
       (effects (font (size 1.27 1.27)))
     )

Commit message: fix boards
Parts:
- added J4: Light jumper, Connector_PinHeader_2.54mm:PinHeader_1x02_P2.54mm_Vertical, symbol Connector_Generic:Conn_01x02
Connections:
- net at J2.4 (Pin_4), J3.1 (Pin_1), U1.4 (OUT): now also J4.1 (Pin_1)
- net at J3.2 (Pin_2), R5.1, R6.1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: now also J4.2 (Pin_2)
Changed lines of the file:
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@@
 (kicad_sch (version 20230121) (generator eeschema)
   (paper "A4")
+  (junction (at 160.02 24.13) (diameter 0) (color 0 0 0 0)
+  )
   (junction (at 120.65 72.39) (diameter 0) (color 0 0 0 0)
   )
@@
   )
   (junction (at 129.54 35.56) (diameter 0) (color 0 0 0 0)
+  )
+  (junction (at 160.02 19.05) (diameter 0) (color 0 0 0 0)
   )
   (junction (at 160.02 50.8) (diameter 0) (color 0 0 0 0)
@@
     (stroke (width 0) (type default))
   )
+  (wire (pts (xy 160.02 24.13) (xy 160.02 27.94))
+    (stroke (width 0) (type default))
+  )
   (wire (pts (xy 66.04 30.48) (xy 69.85 30.48))
     (stroke (width 0) (type default))
   )
+  (wire (pts (xy 184.15 15.24) (xy 160.02 15.24))
+    (stroke (width 0) (type default))
+  )
   (wire (pts (xy 184.15 35.56) (xy 172.72 35.56))
     (stroke (width 0) (type default))
@@
     (stroke (width 0) (type default))
   )
+  (wire (pts (xy 184.15 19.05) (xy 184.15 15.24))
+    (stroke (width 0) (type default))
+  )
+  (wire (pts (xy 160.02 19.05) (xy 129.54 19.05))
+    (stroke (width 0) (type default))
+  )
   (wire (pts (xy 55.88 48.26) (xy 58.42 48.26))
     (stroke (width 0) (type default))
@@
     (stroke (width 0) (type default))
   )
-  (wire (pts (xy 160.02 21.59) (xy 160.02 27.94))
+  (wire (pts (xy 160.02 21.59) (xy 160.02 24.13))
     (stroke (width 0) (type default))
   )
@@
     (stroke (width 0) (type default))
   )
-  (wire (pts (xy 162.56 19.05) (xy 129.54 19.05))
+  (wire (pts (xy 162.56 19.05) (xy 160.02 19.05))
     (stroke (width 0) (type default))
   )
@@
     (stroke (width 0) (type default))
   )
+  (wire (pts (xy 184.15 21.59) (xy 184.15 24.13))
+    (stroke (width 0) (type default))
+  )
   (wire (pts (xy 92.71 64.77) (xy 105.41 64.77))
     (stroke (width 0) (type default))
@@
     (stroke (width 0) (type default))
   )
+  (wire (pts (xy 160.02 15.24) (xy 160.02 19.05))
+    (stroke (width 0) (type default))
+  )
   (wire (pts (xy 172.72 35.56) (xy 172.72 33.02))
     (stroke (width 0) (type default))
@@
   )
   (wire (pts (xy 170.18 38.1) (xy 184.15 38.1))
+    (stroke (width 0) (type default))
+  )
+  (wire (pts (xy 160.02 24.13) (xy 184.15 24.13))
     (stroke (width 0) (type default))
   )
@@
         )
       )
+    )
+  )
+  (symbol (lib_id "Connector_Generic:Conn_01x02") (at 189.23 19.05 0) (unit 1)
+    (in_bom yes) (on_board yes) (dnp no) (fields_autoplaced)
+    (property "Reference" "J4" (at 191.77 19.685 0)
+      (effects (font (size 1.27 1.27)) (justify left))
+    )
+    (property "Value" "Light jumper" (at 191.77 22.225 0)
+      (effects (font (size 1.27 1.27)) (justify left))
+    )
+    (property "Footprint" "Connector_PinHeader_2.54mm:PinHeader_1x02_P2.54mm_Vertical" (at 189.23 19.05 0)
+      (effects (font (size 1.27 1.27)) hide)
+    )
+    (property "Datasheet" "~" (at 189.23 19.05 0)
+      (effects (font (size 1.27 1.27)) hide)
+    )
+    (pin "1")
+    (pin "2")
+    (instances
+      (project "hajo_idealisdioda"
+        (path "/900bec57-3a0d-41dc-a45c-3ae29a4b144e"
+          (reference "J4") (unit 1)
+        )
+      )
