File: hajo/kicad/hajo_kijelzo/hajo_kijelzo.kicad_pcb (KiCad board)
At the start: 2 copper layers, 62 x 92 mm, 21 parts, among them J1 SeaTalk NG, J2 Debug, J3 Fuel, J5 Water, J6 Display, Q1 BC557, U1 MCP2562, U2 LF50CV, U3 LF33_TO220, U4 WeMos_S2_mini

Commit message: pcb plot changes
Parts:
- moved J6 1.55 mm to (26.2, 69.4)
- moved J3 1.53 mm to (23.7, 39.3)
- moved J5 1.52 mm to (23.7, 51.4)
Routing:
- net /T_CS: track 57.6 -> 59.3 mm
- net /SDI: track 61.2 -> 62.8 mm
- net /T_IRQ: track 54.0 -> 55.7 mm
- net /SDO: track 68.8 -> 70.4 mm
- net /L_RESET: track 57.6 -> 59.3 mm
- net /L_DC: track 57.6 -> 59.3 mm
- net /L_CS: track 57.6 -> 59.3 mm
- net /L_BACK: track 32.7 -> 34.3 mm
- net /ADC1_H: track 34.7 -> 36.3 mm
- net /ADC1_L: track 33.3 -> 34.9 mm
- net /Water4: track 32.8 -> 34.3 mm
- net /Water3: track 29.9 -> 31.4 mm
- net /Water1: track 32.3 -> 33.8 mm
- net /Water0: track 33.6 -> 35.1 mm
- net /Water2: track 34.2 -> 35.7 mm
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Other:
- board size 62 x 92 mm -> 65 x 92 mm
