File: hajo/kicad/hajo_kijelzo/hajo_kijelzo.kicad_pcb (KiCad board)
At the start: 2 copper layers, 65 x 92 mm, 21 parts, among them J1 SeaTalk NG, J2 Debug, J3 Fuel, J5 Water, J6 Display, Q1 BC557, U1 MCP2562, U2 LF50CV, U3 LF33_TO220, U4 WeMos_S2_mini

Commit message: amend & upgrade pcbs
Parts:
- added R3: 10K, Resistor_THT:R_Axial_DIN0207_L6.3mm_D2.5mm_P7.62mm_Horizontal, F.Cu at (40.4, 64.1)
- Q1: footprint Package_TO_SOT_THT:TO-92_Inline_Wide -> Package_TO_SOT_THT:TO-92_Inline
- U1: footprint Package_DIP:DIP-8_W7.62mm_Socket -> Package_DIP:DIP-8_W7.62mm
- U4: footprint own:WEMOS_S2_mini_traced -> own:WEMOS_S2_mini
- moved Q1 3.66 mm to (35.1, 62.5)
Connections:
- J2 pad 2: unconnected-(J2-Pin_2-Pad2) -> GND
Routing:
- net /CanStby: track 64.1 -> 81.8 mm
- net +3.3V: track 85.6 -> 100.9 mm
- net GND: track 274.9 -> 285.5 mm
- net /L_BACK: track 34.3 -> 30.8 mm
- net Net-(Q1-B): track 6.91 -> 10.2 mm
Other:
- board text removed: "NC"

Commit message: update existing pcbs
Parts:
- removed J2: Debug, Connector_PinHeader_2.54mm:PinHeader_1x04_P2.54mm_Vertical
- J1: footprint Connector_PinHeader_2.54mm:PinHeader_1x04_P2.54mm_Vertical -> Connector_JST:JST_XH_B4B-XH-A_1x04_P2.50mm_Vertical
- moved J1 1.44 mm to (40.2, 79.9), turned to -90 degrees
Connections:
- U4 pad 16: /DebugTX -> unconnected-(U4-GPIO39-Pad16)
- U4 pad 32: /DebugRX -> unconnected-(U4-GPIO40-Pad32)
Routing:
- net GND: track 285.5 -> 232.4 mm
- net /DebugRX: track 30.3 -> 0.00 mm
- net /DebugTX: track 28.0 -> 0.00 mm
- net /CANL: track 13.5 -> 14.9 mm
- net /CANH: track 9.89 -> 11.3 mm
- net +12V: track 25.6 -> 24.3 mm
Other:
- board text removed: "RXD"
- board text removed: "TXD"
