File: ontozo/kicad/vezerlo/vezerlo.kicad_pcb (KiCad board)
At the start: 2 copper layers, 62 x 92 mm, 17 parts, among them J1 Conn_01x05_Socket, J2 Conn_01x04_Pin, J3 Conn_01x03_Pin, J4 Conn_01x10_Pin, J5 Conn_01x02_Socket, J6 Conn_01x03_Pin, J7 Conn_01x02_Socket, J8 Conn_01x02_Socket, U1 WeMos_S2_mini

Commit message: continue pcb
Parts:
- J1: value Conn_01x05_Socket -> Levels
- J2: renamed from J4; value Conn_01x10_Pin -> Zones
- J3: value Conn_01x03_Pin -> PumpRefill
- J4: renamed from J6; value Conn_01x03_Pin -> PumpMain
- J6: renamed from J2; value Conn_01x04_Pin -> Debug
- J7: value Conn_01x02_Socket -> Button1
- J8: value Conn_01x02_Socket -> BUtton2
- R1: renamed from R8; value R -> 10K
- R3: renamed from R7; value R -> 10K
- R4: renamed from R9; value R -> 10K
- moved J2 31.7 mm to (38.9, 58.5)
- moved R1 28.2 mm to (41.7, 38.1)
- moved J1 20.8 mm to (25.4, 38.1), turned to -90 degrees
- moved R2 19.3 mm to (41.7, 43.2)
- moved R4 17.4 mm to (41.7, 53.4)
- moved R3 10.6 mm to (41.7, 48.3)
- moved J8 6.65 mm to (25.4, 76.5), turned to -90 degrees
- moved J5 6.15 mm to (25.4, 64.8), turned to -90 degrees
- moved J7 5.89 mm to (25.4, 88.4), turned to -90 degrees
- renumbered R6 to R2
Connections:
- net /PumpIrrigate renamed /PumpMain
- net /PumpLift renamed /PumpRefill
Routing:
- net /Level4: track 0.00 -> 34.5 mm
- net /Level1: track 0.00 -> 34.2 mm
- net /Level2: track 0.00 -> 33.1 mm
- net /Level3: track 0.00 -> 29.9 mm
- net +5V: track 29.7 -> 0.00 mm
- net /Zone6: track 0.00 -> 28.2 mm
- net /Zone8: track 0.00 -> 27.2 mm
- net /Zone7: track 0.00 -> 26.2 mm
- net /Zone4: track 0.00 -> 25.5 mm
- net /Zone2: track 0.00 -> 24.2 mm
- net /Zone5: track 0.00 -> 23.5 mm
- net /Zone3: track 0.00 -> 21.7 mm
- net /Zone1: track 0.00 -> 20.7 mm
- net GND: track 66.0 -> 49.4 mm
- net +3.3V: track 0.00 -> 15.2 mm
