File: ontozo/kicad/vezerlo/vezerlo.kicad_pcb (KiCad board)
At the start: 2 copper layers, 62 x 92 mm, 17 parts, among them J1 Levels, J2 Zones, J3 PumpRefill, J4 PumpMain, J5 Conn_01x02_Socket, J6 Debug, J7 Button1, J8 BUtton2, U1 WeMos_S2_mini

Commit message: pcb production
Parts:
- added J10: Zones 9-16, Connector_PinHeader_2.54mm:PinHeader_1x10_P2.54mm_Vertical, F.Cu at (41.8, 85.1)
- J2: value Zones -> Zones 1-8
- J5: value Conn_01x02_Socket -> PowerIn
- J7: value Button1 -> Btn1
- J8: value BUtton2 -> Btn2
- R2: value R -> 10K
- U1: footprint own:WEMOS_S2_mini_traced -> own:WEMOS_S2_mini_gogo
- moved J3 69.0 mm to (41.5, 25.8)
- moved J4 58.1 mm to (53.8, 25.5)
- moved R4 20.2 mm to (45.8, 33.6)
- moved R3 11.1 mm to (45.9, 38.0)
- moved R1 10.4 mm to (46.0, 47.6)
- moved H4 6.79 mm to (77.1, 107.7)
- moved H1 6.08 mm to (25.0, 25.0)
- moved H2 6.08 mm to (25.0, 107.0)
- moved H3 6.08 mm to (77.0, 25.0)
- moved J8 5.30 mm to (27.3, 81.5)
- moved J2 5.17 mm to (41.5, 54.0)
- moved J7 5.16 mm to (27.3, 93.3)
- moved U1 5.11 mm to (55.6, 39.0)
- moved R2 4.34 mm to (46.0, 42.8)
- moved J1 2.90 mm to (27.0, 35.7)
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Connections:
- J1 pad 1: /Level1 -> GND
- J1 pad 2: /Level2 -> /Level1
- J1 pad 3: /Level3 -> /Level2
- J1 pad 4: /Level4 -> /Level3
- J1 pad 5: GND -> /Level4
- J3 pad 1: /PumpRefill -> GND
- J3 pad 3: GND -> /PumpRefill
- J4 pad 1: /PumpMain -> GND
- J4 pad 3: GND -> /PumpMain
- J7 pad 1: /Button1 -> GND
- J7 pad 2: GND -> /Button1
- J8 pad 1: /Button2 -> GND
- J8 pad 2: GND -> /Button2
- R1 pad 2: /Level1 -> /Level4
- R2 pad 2: /Level2 -> /Level3
- R3 pad 2: /Level3 -> /Level2
- R4 pad 2: /Level4 -> /Level1
- U1 pad 11: unconnected-(U1-GPIO16-Pad11) -> /Zone16
- U1 pad 12: unconnected-(U1-GPIO18-Pad12) -> /Zone14
- U1 pad 13: unconnected-(U1-GPIO33-Pad13) -> /Zone12
- U1 pad 14: unconnected-(U1-GPIO35-Pad14) -> /Zone10
- U1 pad 17: /Level1 -> /Zone1
- U1 pad 18: /Level2 -> /Zone2
- U1 pad 19: /Level4 -> /Zone3
- U1 pad 2: /Level3 -> /Level1
- U1 pad 20: /Zone2 -> /Zone4
- U1 pad 21: /Zone4 -> /Zone5
- U1 pad 22: /Zone6 -> /Zone7
- U1 pad 23: /Button1 -> /Button2
- U1 pad 24: /Button2 -> /Button1
- U1 pad 27: unconnected-(U1-GPIO17-Pad27) -> /Zone15
- U1 pad 28: unconnected-(U1-GPIO21-Pad28) -> /Zone13
- U1 pad 29: unconnected-(U1-GPIO34-Pad29) -> /Zone11
- U1 pad 3: /Zone1 -> /Level2
- U1 pad 30: unconnected-(U1-GPIO36-Pad30) -> /Zone9
- U1 pad 4: /Zone3 -> /Level3
- U1 pad 5: /Zone5 -> /Level4
- U1 pad 6: /Zone7 -> /Zone6
Routing:
- net +5V: track 0.00 -> 155.4 mm
- net GND: track 49.4 -> 186.5 mm
- net /Zone16: track 0.00 -> 68.9 mm
- net /Zone14: track 0.00 -> 67.4 mm
- net /Zone15: track 0.00 -> 65.3 mm
- net /Zone12: track 0.00 -> 64.9 mm
- net /Zone13: track 0.00 -> 62.8 mm
- net /Zone10: track 0.00 -> 62.3 mm
- net /Zone11: track 0.00 -> 60.2 mm
- net /Zone9: track 0.00 -> 57.7 mm
- net /Button1: track 0.00 -> 54.4 mm
- net /Button2: track 0.00 -> 49.3 mm
- net /PumpRefill: track 0.00 -> 46.2 mm
- net +3.3V: track 15.2 -> 57.0 mm
- net /PumpMain: track 0.00 -> 36.3 mm
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Other:
- outline, holes or cut-outs redrawn
- board text added: "+5V"
- board text added: "1"
- board text added: "12"
- board text added: "13"
- board text added: "16"
- board text added: "4"
- board text added: "5"
- board text added: "8"
- board text added: "9"

Commit message: pcb led light for buttons
Parts:
- removed J7: Btn1, TerminalBlock_Phoenix:TerminalBlock_Phoenix_MKDS-1,5-2-5.08_1x02_P5.08mm_Horizontal
- removed J8: Btn2, TerminalBlock_Phoenix:TerminalBlock_Phoenix_MKDS-1,5-2-5.08_1x02_P5.08mm_Horizontal
- added J11: Btn2, TerminalBlock_Phoenix:TerminalBlock_Phoenix_MKDS-1,5-4-5.08_1x04_P5.08mm_Horizontal, F.Cu at (27.5, 61.4)
- added J9: Btn1, TerminalBlock_Phoenix:TerminalBlock_Phoenix_MKDS-1,5-4-5.08_1x04_P5.08mm_Horizontal, F.Cu at (27.4, 84.0)
- added RV1: 10k, Potentiometer_THT:Potentiometer_Bourns_3386P_Vertical, F.Cu at (39.3, 70.5)
- added RV2: 10k, Potentiometer_THT:Potentiometer_Bourns_3386P_Vertical, F.Cu at (39.1, 92.7)
- moved J5 39.8 mm to (36.7, 105.4), turned to 0 degrees
- moved J10 8.18 mm to (49.6, 82.7)
- moved J2 7.89 mm to (49.4, 53.5)
- moved J1 3.45 mm to (27.1, 32.3)
Connections:
- J5 pad 1: +5V -> GND
- J5 pad 2: GND -> +5V
Routing:
- net GND: track 186.5 -> 270.1 mm
- net Net-(J11-Pin_2): track 0.00 -> 15.0 mm
- net Net-(J9-Pin_2): track 0.00 -> 14.6 mm
- net /Button1: track 54.4 -> 61.7 mm
- net /Zone12: track 64.9 -> 59.2 mm
- net /Zone16: track 68.9 -> 63.3 mm
- net /Zone9: track 57.7 -> 52.1 mm
- net /Zone13: track 62.8 -> 57.2 mm
- net /Zone11: track 60.2 -> 54.6 mm
- net /Zone15: track 65.3 -> 59.7 mm
- net /Zone14: track 67.4 -> 61.7 mm
- net /Zone10: track 62.3 -> 56.7 mm
- net /Zone7: track 28.1 -> 24.2 mm
- net /Zone5: track 25.5 -> 21.7 mm
- net /Zone8: track 25.9 -> 22.2 mm
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Other:
- board text added: "Led+"
- board text added: "Led-"
- board text added: "Out"
- board text added: "Switch"
