File: ontozo/kicad/vezerlo/vezerlo.kicad_sch (KiCad schematic)
At the start: 17 parts, among them J1 Conn_01x05_Socket, J2 Conn_01x04_Pin, J3 Conn_01x03_Pin, J4 Conn_01x10_Pin, J5 Conn_01x02_Socket, J6 Conn_01x03_Pin, J7 Conn_01x02_Socket, J8 Conn_01x02_Socket, U1 WeMos_S2_mini

Commit message: continue pcb
Parts:
- J1: value Conn_01x05_Socket -> Levels
- J2: renamed from J4; value Conn_01x10_Pin -> Zones
- J3: value Conn_01x03_Pin -> PumpRefill
- J4: renamed from J6; value Conn_01x03_Pin -> PumpMain
- J6: renamed from J2; value Conn_01x04_Pin -> Debug
- J7: value Conn_01x02_Socket -> Button1
- J8: value Conn_01x02_Socket -> BUtton2
- R1: renamed from R8; value R -> 10K
- R3: renamed from R7; value R -> 10K
- R4: renamed from R9; value R -> 10K
- renumbered R6 to R2
Connections:
- net PumpIrrigate renamed PumpMain
- net PumpLift renamed PumpRefill
Changed lines of the file:
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@@
 		)
 	)
-	(label "PumpLift"
+	(label "PumpRefill"
 		(at 151.13 74.93 0)
 		(fields_autoplaced yes)
@@
 		)
 	)
-	(label "PumpIrrigate"
+	(label "PumpMain"
 		(at 130.81 71.12 180)
 		(fields_autoplaced yes)
@@
 		)
 	)
-	(label "PumpLift"
+	(label "PumpRefill"
 		(at 130.81 90.17 180)
 		(fields_autoplaced yes)
@@
 		)
 	)
-	(label "PumpIrrigate"
+	(label "PumpMain"
 		(at 151.13 72.39 0)
 		(fields_autoplaced yes)
@@
 		(on_board yes)
 		(dnp no)
-		(property "Reference" "R9"
+		(property "Reference" "R4"
 			(at 105.41 54.61 90)
 			(effects
@@
 			)
 		)
-		(property "Value" "R"
+		(property "Value" "10K"
 			(at 105.41 49.53 90)
 			(effects
@@
 			(project "vezerlo"
 				(path "/900bec57-3a0d-41dc-a45c-3ae29a4b144e"
-					(reference "R9")
+					(reference "R4")
 					(unit 1)
 				)
@@
 			)
 		)
-		(property "Value" "Conn_01x03_Pin"
+		(property "Value" "PumpRefill"
 			(at 109.855 87.63 0)
 			(effects
@@
 		(on_board yes)
 		(dnp no)
-		(property "Reference" "R7"
+		(property "Reference" "R3"
 			(at 105.41 45.72 90)
 			(effects
@@
 			)
 		)
-		(property "Value" "R"
+		(property "Value" "10K"
 			(at 105.41 40.64 90)
 			(effects
@@
 			(project "vezerlo"
 				(path "/900bec57-3a0d-41dc-a45c-3ae29a4b144e"
-					(reference "R7")
+					(reference "R3")
 					(unit 1)
 				)
@@
 			)
 		)
-		(property "Value" "Conn_01x02_Socket"
+		(property "Value" "Button1"
 			(at 26.67 73.6599 0)
 			(effects
@@
 		(on_board yes)
 		(dnp no)
-		(property "Reference" "R6"
+		(property "Reference" "R2"
 			(at 105.41 36.83 90)
 			(effects
@@
 			(project "vezerlo"
 				(path "/900bec57-3a0d-41dc-a45c-3ae29a4b144e"
-					(reference "R6")
+					(reference "R2")
 					(unit 1)
 				)
@@
 		(on_board yes)
 		(dnp no)
-		(property "Reference" "J2"
+		(property "Reference" "J6"
 			(at 35.56 27.305 0)
 			(effects
@@
 			)
 		)
-		(property "Value" "Conn_01x04_Pin"
+		(property "Value" "Debug"
 			(at 35.56 24.765 0)
 			(effects
@@
 			(project "vezerlo"
 				(path "/900bec57-3a0d-41dc-a45c-3ae29a4b144e"
-					(reference "J2")
+					(reference "J6")
 					(unit 1)
 				)
@@
 		(on_board yes)
 		(dnp no)
-		(property "Reference" "J6"
+		(property "Reference" "J4"
 			(at 109.855 66.04 0)
 			(effects
@@
 			)
 		)
-		(property "Value" "Conn_01x03_Pin"
+		(property "Value" "PumpMain"
 			(at 109.855 68.58 0)
 			(effects
@@
 			(project "vezerlo"
 				(path "/900bec57-3a0d-41dc-a45c-3ae29a4b144e"
-					(reference "J6")
+					(reference "J4")
 					(unit 1)
 				)
@@
 			)
 		)
-		(property "Value" "Conn_01x05_Socket"
+		(property "Value" "Levels"
 			(at 75.565 29.21 0)
 			(effects
@@
 		(on_board yes)
 		(dnp no)
-		(property "Reference" "J4"
+		(property "Reference" "J2"
 			(at 81.915 97.79 0)
 			(effects
@@
 			)
 		)
-		(property "Value" "Conn_01x10_Pin"
+		(property "Value" "Zones"
 			(at 81.915 95.25 0)
 			(effects
@@
 			(project ""
 				(path "/900bec57-3a0d-41dc-a45c-3ae29a4b144e"
-					(reference "J4")
+					(reference "J2")
 					(unit 1)
 				)
@@
 			)
 		)
-		(property "Value" "Conn_01x02_Socket"
+		(property "Value" "BUtton2"
 			(at 26.67 86.3599 0)
 			(effects
@@
 		(on_board yes)
 		(dnp no)
-		(property "Reference" "R8"
+		(property "Reference" "R1"
 			(at 105.41 29.21 90)
 			(effects
@@
 			)
 		)
-		(property "Value" "R"
+		(property "Value" "10K"
 			(at 105.41 24.13 90)
 			(effects
@@
 			(project "vezerlo"
 				(path "/900bec57-3a0d-41dc-a45c-3ae29a4b144e"
-					(reference "R8")
-					(unit 1)
-				)
+					(reference "R1")
+					(unit 1)
+				)
