File: ontozo/kicad/vezerlo/vezerlo.kicad_sch (KiCad schematic)
At the start: 17 parts, among them J1 Levels, J2 Zones, J3 PumpRefill, J4 PumpMain, J5 Conn_01x02_Socket, J6 Debug, J7 Button1, J8 BUtton2, U1 WeMos_S2_mini

Commit message: pcb kickoff
Parts:
- J5: value Conn_01x02_Socket -> PowerIn
- J7: value Button1 -> Btn1
- J8: value BUtton2 -> Btn2
- R2: value R -> 10K
Other:
- moved on the sheet: J1, J6, R1, R2, R3, R4

Commit message: pcb production
Parts:
- added J10: Zones 9-16, Connector_PinHeader_2.54mm:PinHeader_1x10_P2.54mm_Vertical, symbol Connector:Conn_01x10_Pin
- J2: value Zones -> Zones 1-8
- U1: footprint own:WEMOS_S2_mini_traced -> own:WEMOS_S2_mini_gogo
Connections:
- net +5V: now also J10.10 (Pin_10)
- net Button1: now also J7.2 (Pin_2), U1.24 (GPIO14); no longer J7.1 (Pin_1), U1.23 (GPIO13)
- net Button2: now also J8.2 (Pin_2), U1.23 (GPIO13); no longer J8.1 (Pin_1), U1.24 (GPIO14)
- net GND: now also J1.1 (Pin_1), J3.1 (Pin_1), J4.1 (Pin_1), J7.1 (Pin_1), J8.1 (Pin_1), J10.1 (Pin_1); no longer J1.5 (Pin_5), J3.3 (Pin_3), J4.3 (Pin_3), J7.2 (Pin_2), J8.2 (Pin_2)
- net Level1: now also J1.2 (Pin_2), R4.2, U1.2 (GPIO3); no longer J1.1 (Pin_1), R1.2, U1.17 (GPIO1)
- net Level2: now also J1.3 (Pin_3), R3.2, U1.3 (GPIO5); no longer J1.2 (Pin_2), R2.2, U1.18 (GPIO2)
- net Level3: now also J1.4 (Pin_4), R2.2, U1.4 (GPIO7); no longer J1.3 (Pin_3), R3.2, U1.2 (GPIO3)
- net Level4: now also J1.5 (Pin_5), R1.2, U1.5 (GPIO9); no longer J1.4 (Pin_4), R4.2, U1.19 (GPIO4)
- net PumpMain: now also J4.3 (Pin_3); no longer J4.1 (Pin_1)
- net PumpRefill: now also J3.3 (Pin_3); no longer J3.1 (Pin_1)
- net Zone1: now also U1.17 (GPIO1); no longer U1.3 (GPIO5)
- net Zone2: now also U1.18 (GPIO2); no longer U1.20 (GPIO6)
- net Zone3: now also U1.19 (GPIO4); no longer U1.4 (GPIO7)
- net Zone4: now also U1.20 (GPIO6); no longer U1.21 (GPIO8)
- net Zone5: now also U1.21 (GPIO8); no longer U1.5 (GPIO9)
- net Zone6: now also U1.6 (GPIO11); no longer U1.22 (GPIO10)
- net Zone7: now also U1.22 (GPIO10); no longer U1.6 (GPIO11)
- net Zone16: now reaches U1.11 (GPIO16)
- net Zone16: now also J10.9 (Pin_9)
- net Zone14: now reaches U1.12 (GPIO18)
- net Zone14: now also J10.7 (Pin_7)
- net Zone12: now reaches U1.13 (GPIO33)
- net Zone12: now also J10.5 (Pin_5)
- net Zone10: now reaches U1.14 (GPIO35)
- net Zone10: now also J10.3 (Pin_3)
- net Zone15: now reaches U1.27 (GPIO17)
- net Zone15: now also J10.8 (Pin_8)
- net Zone13: now reaches U1.28 (GPIO21)
- net Zone13: now also J10.6 (Pin_6)
- net Zone11: now reaches U1.29 (GPIO34)
- net Zone11: now also J10.4 (Pin_4)
- net Zone9: now reaches U1.30 (GPIO36)
- net Zone9: now also J10.2 (Pin_2)
- no-connect marks 11 -> 3
Other:
- moved on the sheet: J1, J3, J6, J7, J8

Commit message: pcb led light for buttons
Parts:
- removed J7: Btn1, TerminalBlock_Phoenix:TerminalBlock_Phoenix_MKDS-1,5-2-5.08_1x02_P5.08mm_Horizontal, symbol Connector:Conn_01x02_Socket
- removed J8: Btn2, TerminalBlock_Phoenix:TerminalBlock_Phoenix_MKDS-1,5-2-5.08_1x02_P5.08mm_Horizontal, symbol Connector:Conn_01x02_Socket
- added J11: Btn2, TerminalBlock_Phoenix:TerminalBlock_Phoenix_MKDS-1,5-4-5.08_1x04_P5.08mm_Horizontal, symbol Connector:Conn_01x04_Pin
- added J9: Btn1, TerminalBlock_Phoenix:TerminalBlock_Phoenix_MKDS-1,5-4-5.08_1x04_P5.08mm_Horizontal, symbol Connector:Conn_01x04_Pin
- added RV1, RV2: 10k, Potentiometer_THT:Potentiometer_Bourns_3386P_Vertical, symbol Device:R_Potentiometer
Connections:
- net +5V: now also J5.2 (Pin_2), RV1.1, RV2.1; no longer J5.1 (Pin_1)
- net Button1: now also J9.4 (Pin_4)
- net Button2: now also J11.4 (Pin_4)
- net GND: now also J5.1 (Pin_1), J11.1 (Pin_1), J11.3 (Pin_3), J9.1 (Pin_1), J9.3 (Pin_3); no longer J5.2 (Pin_2)
- new net: J11.2 (Pin_2), RV1.2
- new net: J9.2 (Pin_2), RV2.2
- no-connect marks 3 -> 5
Other:
- moved on the sheet: J5
