File: hajo/kicad/hajo_akku/hajo_akku.kicad_sch (KiCad schematic)
At the start: 21 parts, among them J1 Seetalk NG, J2 Debug, J3 Batteries, U1 MCP2562, U2 LF50CV, U3 WeMos_S2_mini

Commit message: amend & upgrade pcbs
Parts:
- added C6: 100n, Capacitor_THT:C_Rect_L7.0mm_W2.0mm_P5.00mm, symbol Device:C
- added C7: 2.2u, Capacitor_THT:CP_Radial_D5.0mm_P2.00mm, symbol Device:C_Polarized
- added U4: LF33, Package_TO_SOT_THT:TO-220-3_Vertical, symbol Regulator_Linear:LF50_TO220
- U1: footprint Package_DIP:DIP-8_W7.62mm_Socket -> Package_DIP:DIP-8_W7.62mm
- U2: value LF50CV -> LF50
- U3: footprint own:WEMOS_S2_mini_traced -> own:WEMOS_S2_mini
Connections:
- net +3.3V: now also C7.1, U4.3 (VO)
- net +5V: now also C6.1, U4.1 (VI)
- net GND: now also J2.2 (Pin_2), C6.2, C7.2, U4.2 (GND)
- no-connect marks 20 -> 19
Other:
- moved on the sheet: J1

Commit message: update existing pcbs
Parts:
- removed J2: Debug, Connector_PinHeader_2.54mm:PinHeader_1x04_P2.54mm_Vertical, symbol Connector:Conn_01x04_Pin
- J1: footprint Connector_PinHeader_2.54mm:PinHeader_1x04_P2.54mm_Vertical -> Connector_JST:JST_XA_B04B-XASK-1_1x04_P2.50mm_Vertical
- J3: footprint Connector_PinHeader_2.54mm:PinHeader_1x03_P2.54mm_Vertical -> Connector_JST:JST_XH_B3B-XH-A_1x03_P2.50mm_Vertical
Connections:
- net DebugRX: no longer names the net of U3.32 (GPIO40)
- net DebugTX: no longer names the net of U3.16 (GPIO39)
- no-connect marks 19 -> 21

Commit message: redesign akku pcb
Parts:
- removed C2, C6: 100n, Capacitor_THT:C_Rect_L7.0mm_W2.0mm_P5.00mm, symbol Device:C
Connections:
- net +5V: no longer U3.9 (VBUS)
- net CANH: now also J1.2 (Pin_2); no longer J1.3 (Pin_3)
- net CANL: now also J1.3 (Pin_3); no longer J1.4 (Pin_4)
- net GND: now also J1.4 (Pin_4), U1.8 (STBY); no longer J1.2 (Pin_2)
- net CanStby: no longer names the net of U3.22 (GPIO10)
- net CanStby: no longer U1.8 (STBY)
- no-connect marks 21 -> 23
